Commit message: final version thesis

File: urdf/robocol_arm.urdf (robot description, URDF)
Before this commit: robot robocol_arm, 7 links, 6 joints
Joints:
- joint robocol_joint1: limit lower=-2.09 upper=2.09 effort=87 velocity=2.3925 -> lower=-1.5708 upper=1.2217 effort=87 velocity=2.3925
- joint robocol_joint2: limit lower=-2.75 upper=2.75 effort=87 velocity=2.3925 -> lower=-1.7453 upper=2.3562 effort=87 velocity=2.3925
- joint robocol_joint3: limit lower=-2.87 upper=2.76 effort=87 velocity=2.3925 -> lower=-2.4435 upper=2.5307 effort=87 velocity=2.3925
- joint robocol_joint5: limit lower=-2.39 upper=2.7 effort=12 velocity=2.8710 -> lower=-2.39 upper=2.39 effort=12 velocity=2.8710
- joint robocol_joint6: limit lower=-2.97 upper=2.97 effort=12 velocity=2.8710 -> lower=-6.28 upper=6.28 effort=12 velocity=2.8710
